Commit message: Add files via upload

File: ackermann_vehicle_description/urdf/em_3905.urdf.xacro (robot description, xacro)
@@ -321,7 +321,7 @@
       <origin xyz="0 0 ${-chassis_height / 2}"/>
       <geometry>
-        <mesh
-          filename="package://ackermann_vehicle_description/meshes/base_link.STL"/>
-        <!--box size="${chassis_length} ${chassis_width} ${chassis_height}"/-->
+        <!--mesh
+          filename="package://ackermann_vehicle_description/meshes/base_link.STL"/-->
+        <box size="${chassis_length} ${chassis_width} ${chassis_height}"/>
       </geometry>
       <material name="chassis_mat"/>
@@ -330,6 +330,6 @@
       <origin xyz="0 0 ${-chassis_height / 2}"/>
       <geometry>
-        <filename="package://ackermann_vehicle_description/meshes/base_link.STL"/>
-        <!--box size="${chassis_length} ${chassis_width} ${chassis_height}"/-->
+        <!--filename="package://ackermann_vehicle_description/meshes/base_link.STL"/-->
+        <box size="${chassis_length} ${chassis_width} ${chassis_height}"/>
       </geometry>
     </collision>
@@ -348,9 +348,9 @@
         izz="0.00338508790406167" />
     </inertial>
-    <!--xacro:solid_cuboid_inertial
+    <xacro:solid_cuboid_inertial
         width="${chassis_length}" depth="${chassis_width}"
         height="${chassis_height}" mass="${chassis_mass}">
       <origin xyz="0 0 ${-chassis_height / 2}"/>
-    </xacro:solid_cuboid_inertial-->
+    </xacro:solid_cuboid_inertial>
   </link>
   <gazebo reference="chassis">
@@ -361,8 +361,8 @@
     <child link="chassis"/>
   </joint>
-  <!-- Batteries >
+  <!--Batteries-->
   <xacro:battery prefix="left" reflect="1"/>
-  <xacro:battery prefix="right" reflect="-1"/-->
-  <!-- Wheels >
+  <xacro:battery prefix="right" reflect="-1"/>
+  <!--Wheels-->
   <xacro:front_wheel lr_prefix="left" fr_prefix="front"
                      lr_reflect="1" fr_reflect="1"/>
@@ -372,5 +372,5 @@
                     lr_reflect="1" fr_reflect="-1"/>
   <xacro:rear_wheel lr_prefix="right" fr_prefix="rear"
-                    lr_reflect="-1" fr_reflect="-1"/-->
+                    lr_reflect="-1" fr_reflect="-1"/>
   <gazebo>
     <plugin name="gazebo_ros_control" filename="libgazebo_ros_control.so"/>
